File: brilliant-button-breakout-board.kicad_pcb (KiCad board)
At the start: 2 copper layers, 38.6 x 15.7 mm, 12 parts, among them J1 Conn_01x03, J2 Conn_01x03, J3 Conn_01x03, J4 Conn_01x03, SW1 SW_Push, SW2 SW_Push, SW3 SW_Push, SW4 SW_Push

Commit message: capacitor update
Parts:
- added C1: C, Capacitor_SMD:C_0603_1608Metric_Pad1.05x0.95mm_HandSolder, B.Cu at (105.2, 73.4)
- added C2: C, Capacitor_SMD:C_0603_1608Metric_Pad1.05x0.95mm_HandSolder, B.Cu at (105.2, 74.9)
- added C3: C, Capacitor_SMD:C_0603_1608Metric_Pad1.05x0.95mm_HandSolder, B.Cu at (115.6, 73.4)
- added C4: C, Capacitor_SMD:C_0603_1608Metric_Pad1.05x0.95mm_HandSolder, B.Cu at (115.6, 74.9)
- added C5: C, Capacitor_SMD:C_0603_1608Metric_Pad1.05x0.95mm_HandSolder, B.Cu at (125.5, 73.4)
- added C6: C, Capacitor_SMD:C_0603_1608Metric_Pad1.05x0.95mm_HandSolder, B.Cu at (125.5, 74.9)
- added C7: C, Capacitor_SMD:C_0603_1608Metric_Pad1.05x0.95mm_HandSolder, B.Cu at (135.6, 73.4)
- added C8: C, Capacitor_SMD:C_0603_1608Metric_Pad1.05x0.95mm_HandSolder, B.Cu at (135.6, 74.9)
- R1, R2, R3, R4: moved to B.Cu
- moved R2 6.51 mm to (119.1, 74.2), turned to 90 degrees
- moved R3 6.51 mm to (129.3, 74.2), turned to 90 degrees
- moved R4 6.51 mm to (139.4, 74.2), turned to 90 degrees
- moved R1 6.51 mm to (109.0, 74.2), turned to 90 degrees
Routing:
- net Net-(C2-Pad1): track 83.3 -> 102.5 mm
- net Net-(C1-Pad2): track 102.1 -> 116.1 mm
- net Net-(C7-Pad1): track 14.7 -> 19.1 mm
- net Net-(C5-Pad1): track 14.7 -> 19.1 mm
- net Net-(C1-Pad1): track 14.7 -> 19.1 mm
- net Net-(C3-Pad1): track 14.7 -> 18.9 mm
Other:
- board size 38.6 x 15.7 mm -> 38.6 x 14.5 mm
- board text removed: "10k"
